File: rf-dongle.kicad_pcb (KiCad board)
At the start: 4 copper layers, 25.3 x 29.6 mm, 30 parts, among them J1 USB_A, J2 TC2030, SW1 SW_Push, U1 NRF52840-QIAA-F-R, X1 32MHz

Commit message: ordered rev 2
Routing:
- net GND: track 41.7 -> 42.3 mm
Other:
- board text removed: "TODO double check: - RF impedance 50 ohm - USB data impedance 90 ohm REDO silkscreen"
Changed lines of the file:
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@@
 	)
 	(gr_rect
-		(start 33.05 38.4)
-		(end 52.3 39.15)
+		(start 33.05 38.25)
+		(end 58.3 39)
 		(stroke
 			(width 0.2)
@@
 	)
 	(gr_rect
-		(start 33 38.425)
-		(end 33.75 41.375)
+		(start 33 38.25)
+		(end 33.75 56.35)
 		(stroke
 			(width 0.2)
@@
 	)
 	(gr_rect
-		(start 32.75 53.575)
-		(end 33.5 56.425)
+		(start 57.5 38.325)
+		(end 58.25 56.425)
 		(stroke
 			(width 0.2)
@@
 	)
 	(gr_rect
-		(start 51.725 38.475)
-		(end 52.475 56.325)
+		(start 46.75 55.875)
+		(end 58.25 56.625)
 		(stroke
 			(width 0.2)
@@
 		(layer "User.1")
 	)
-	(gr_rect
-		(start 33.5 55.5)
-		(end 51.75 56.25)
-		(stroke
-			(width 0.2)
-			(type solid)
-		)
-		(fill yes)
-		(layer "User.1")
-	)
 	(gr_line
 		(start 51.8 36.2)
@@
 		)
 		(layer "User.2")
-	)
-	(gr_poly
-		(pts
-			(xy 19.4625 41.4375) (xy 19.4625 53.4375) (xy 32.9625 53.4375) (xy 32.9625 56.4375) (xy 52.4625 56.4375)
-			(xy 52.4625 38.3875) (xy 32.9625 38.3875) (xy 32.9625 41.4375)
-		)
-		(stroke
-			(width 0.2)
-			(type solid)
-		)
-		(fill no)
-		(layer "User.4")
 	)
 	(gr_text "LED2"
@@
 		)
 	)
-	(gr_text "TODO double check:\n- RF impedance 50 ohm \n- USB data impedance 90 ohm\n\nREDO silkscreen"
-		(at 63.1 60.3 0)
-		(layer "User.2")
-		(effects
-			(font
-				(size 1 1)
-				(thickness 0.15)
-			)
-			(justify left bottom)
-		)
-	)
 	(gr_text "Keepout"
 		(at 53.9 31.8 270)
@@
 	)
 	(segment
-		(start 45.8 39.2)
-		(end 45.8 40.1)
-		(width 0.25)
-		(layer "F.Cu")
-		(net 2)
-	)
-	(segment
 		(start 40.5 45.975)
 		(end 42 47.475)
@@
 		(start 42.25 41.245)
 		(end 42.25 40.45)
+		(width 0.25)
+		(layer "F.Cu")
+		(net 2)
+	)
+	(segment
+		(start 44.75 39.05)
+		(end 45.8 40.1)
 		(width 0.25)
 		(layer "F.Cu")
@@
 	)
 	(via
-		(at 45.8 39.2)
+		(at 44.75 39.05)
 		(size 0.6)
 		(drill 0.3)
